Commit message: trying to fuse lowsate joint info for better odom

File: src/man_mapping/urdf/go2_description.urdf (robot description, URDF)
Before this commit: robot go2_description, 42 links, 41 joints
Links:
- removed link base
- added link base_link, mass 6.921; collision box size=0.3762 0.0935 0.114; visual mesh filename=package://man_mapping/dae/base.dae
Joints:
- joint FL_hip_joint: parent base -> base_link
- joint FL_hip_rotor_joint: parent base -> base_link
- joint FR_hip_joint: parent base -> base_link
- joint FR_hip_rotor_joint: parent base -> base_link
- joint Head_upper_joint: parent base -> base_link
- joint RL_hip_joint: parent base -> base_link
- joint RL_hip_rotor_joint: parent base -> base_link
- joint RR_hip_joint: parent base -> base_link
- joint RR_hip_rotor_joint: parent base -> base_link
- joint front_camera_joint: parent base -> base_link
- joint imu_joint: parent base -> base_link
- joint radar_joint: parent base -> base_link
